File: BSPD SAE.kicad_sch (KiCad schematic)
At the start: 22 parts, among them U1 TLV1842QDGKRQ1, U2 TLV1842QDGKRQ1

Commit message: autosave 2026-09-24 14:46:54
Connections:
- net Vsig1: no longer R6.1
- new net Acc: R6.1
Changed lines of the file:
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@@
 	(generator "eeschema")
 	(generator_version "10.0")
-	(paper "A4")
+	(paper "A3")
 	(text "Comparator used :TLV1842-Q1\n\nTop compares break pedal position and set voltage.\n\nBottom Checks if there is break in the wire/if we are recieving a signal (rule requirement)\n"
 		(exclude_from_sim no)
@@
 		)
 	)
-	(global_label "Vsig1"
+	(global_label "Acc"
 		(shape input)
 		(at 34.29 54.61 180)
@@
 		)
 		(property "Intersheetrefs" "${INTERSHEET_REFS}"
-			(at 26.2248 54.61 0)
+			(at 28.039 54.61 0)
 			(hide yes)
 			(show_name no)

Commit message: autosave 2026-09-29 17:41:24
Parts:
- removed C1, C3: 10uf, Capacitor_SMD:C_1210_3225Metric, symbol Device:C_Small
- removed C2, C4: 100nf, PCM_4ms_Capacitor:C_0603, symbol Device:C_Small
- removed R1, R2, R3, R4: 3296W-1-103LF, POT_3296W, symbol 2026-08-27_05-53-58:3296W-1-103LF
- removed R10, R11, R13, R14, R16, R5, R6, R9: 10k, Resistor_SMD:R_0805_2012Metric, symbol PCM_SparkFun-Resistor:R_Small
- removed R12, R15, R7, R8: 1M, Resistor_SMD:R_0805_2012Metric, symbol PCM_SparkFun-Resistor:R_Small
- removed U1, U2: TLV1842QDGKRQ1, DGK0008A-IPC_A, symbol 2026-08-27_05-25-16:TLV1842QDGKRQ1
- added C5, C7: 10uf, Capacitor_SMD:C_1210_3225Metric, symbol Device:C_Small
- added C6, C8: 100nf, PCM_4ms_Capacitor:C_0603, symbol Device:C_Small
- added C9: 1uf, PCM_4ms_Capacitor:C_0603, symbol Device:C_Small
- added R17, R22, R26, R27, R32, R33: 3296W-1-103LF, POT_3296W, symbol 2026-08-27_05-53-58:3296W-1-103LF
- added R18, R19, R23, R28, R29, R34, R35, R36, R37, R38, R44, R45, R46: 10k, Resistor_SMD:R_0805_2012Metric, symbol PCM_SparkFun-Resistor:R_Small
- added R20, R24, R30, R39, R40, R42: 1M, Resistor_SMD:R_0805_2012Metric, symbol PCM_SparkFun-Resistor:R_Small
- added U3, U4: TLV1824, BSPD:TSSOP-14_4.4x5mm_P0.65mm_TI_PW, symbol TLV1824:TLV1824
Connections:
- net 5V supply: now also R17.1, R22.1, R26.1, R27.1, R32.1, R33.1, R44.2, R45.2, U3.10 (-), U4.10 (-)
- net GND: now also C5.2, C6.2, C7.2, C8.2, C9.1, R17.3, R19.1, R22.3, R26.3, R27.3, R32.3, R33.3, R34.1, U3.11 (+), U3.12 (V-), U4.11 (+), U4.12 (V-)
- net Vsupply12: now also C5.1, C6.1, C7.1, C8.1, U3.3 (V+), U4.3 (V+)
- new net: R28.2, U3.8 (-)
- new net: R33.2, U4.6 (-)
- new net: R38.2, R40.1, U4.7 (+)
- new net: R22.2, U3.6 (-)
- new net: R35.2, U4.8 (-)
- new net: R18.2, R20.1, U3.5 (+)
- new net: R32.2, R36.1
- new net: R36.2, R39.1, U4.9 (+)
- new net: R26.2, U4.4 (-)
- new net: R23.2, R24.1, U3.7 (+)
- new net: R37.2, R42.1, U4.5 (+)
- new net: R29.2, R30.1, U3.9 (+)
- new net: R17.2, U3.4 (-)
- new net: R27.2, R29.1
- new net 5kw level: R18.1, R19.2, R23.1, R28.1
- new net 5kw level demand reached: R20.2, R42.2, R44.1, U3.2, U4.2
- new net Brake Sensor: R34.2, R35.1, R37.1, R38.1
- new net Latch Input Sensor after 10ms: C9.2, R46.1
- new net No fault in sensor wiring: R24.2, R30.2, R39.2, R40.2, R45.1, R46.2, U3.1, U3.14, U4.1, U4.14
- no-connect marks 0 -> 2
Other:
- note added: "Comparator used :TLV1824 Logic explained U3A is what will be used to compare the actual signal level with U4A. If U3A outputs high that means we have reached 5KW demand Per Rule book limits While U3B and U3C are wired the opposite way both will output high if there conditions arent met. when they pull low this indicates a problem with the wiring which will shutdown the car instantly"
- note added: "Comparator used :TLV1824 Logic same as above but U4A measure brake force limits is about 20% look at rule book to confirm Same logic as U3B and C for U4B and C except for Brake force wire"
- note removed: "Comparator used :TLV1842-Q1 Top compares break pedal position and set voltage. Bottom Checks if there is break in the wire/if we are recieving a signal (rule requirement)"

Commit message: autosave 2026-09-30 01:54:18
Parts:
- C6, C8, C9: footprint PCM_4ms_Capacitor:C_0603 -> Capacitor_SMD:C_0805_2012Metric
- C7: footprint Capacitor_SMD:C_1210_3225Metric -> Capacitor_SMD:C_0805_2012Metric
Changed lines of the file:
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@@
 			)
 		)
-		(property "Footprint" "PCM_4ms_Capacitor:C_0603"
+		(property "Footprint" "Capacitor_SMD:C_0805_2012Metric"
 			(at 256.54 222.25 0)
 			(hide yes)
@@
 			)
 		)
-		(property "Footprint" "PCM_4ms_Capacitor:C_0603"
+		(property "Footprint" "Capacitor_SMD:C_0805_2012Metric"
 			(at 148.59 152.4 0)
 			(hide yes)
@@
 			)
 		)
-		(property "Footprint" "Capacitor_SMD:C_1210_3225Metric"
+		(property "Footprint" "Capacitor_SMD:C_0805_2012Metric"
 			(at 138.43 152.4 0)
 			(hide yes)
@@
 			)
 		)
-		(property "Footprint" "PCM_4ms_Capacitor:C_0603"
+		(property "Footprint" "Capacitor_SMD:C_0805_2012Metric"
 			(at 149.86 22.86 0)
 			(hide yes)

Commit message: autosave 2026-09-30 19:58:07
Parts:
- added C11: 100nf, Capacitor_SMD:C_0805_2012Metric, symbol Device:C_Small
- added R1: 1M, symbol Device:R_Small
- added R2: 523k, symbol Device:R_Small
- added R3: 715K, symbol Device:R_Small
- added U1: LTC6994xS6-2, Package_TO_SOT_SMD:TSOT-23-6, symbol Timer:LTC6994xS6-2
Connections:
- net 5V supply: now also C11.1, R1.1, U1.5 (V+)
- net 5kw level demand reached: now also U1.1 (IN)
- net GND: now also C11.2, R2.2, R3.2, U1.2 (GND)
- new net: R1.2, R2.1, U1.4 (DIV)
- new net: R3.1, U1.3 (SET)
- new net Brake_and_5KW_After_Delay: U1.6 (OUT)

Commit message: autosave 2026-09-30 20:02:27
Other:
- note added: "IC Configure tool:https://beta-tools.analog.com/timerblox/LTC6994 delay amount .470s"
Changed lines of the file:
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@@
 	(generator_version "10.0")
 	(paper "A3")
+	(text "IC Configure tool:https://beta-tools.analog.com/timerblox/LTC6994\ndelay amount .470s"
+		(exclude_from_sim no)
+		(at 306.578 22.86 0)
+		(effects
+			(font
+				(size 1.27 1.27)
+			)
+		)
+	)
 	(text "Comparator used :TLV1824\nLogic same as above but U4A measure brake force limits is about 20% look\nat rule book to confirm \n\nSame logic as U3B and C for U4B and C except for Brake force wire"
 		(exclude_from_sim no)

Commit message: autosave 2026-09-30 20:11:07
Parts:
- U3, U4: footprint BSPD:TSSOP-14_4.4x5mm_P0.65mm_TI_PW -> TSSOP-14_4.4x5mm_P0.65mm_TI_PW
Changed lines of the file:
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@@
 			)
 		)
-		(property "Footprint" "BSPD:TSSOP-14_4.4x5mm_P0.65mm_TI_PW"
+		(property "Footprint" "TSSOP-14_4.4x5mm_P0.65mm_TI_PW"
 			(at 157.48 17.78 0)
 			(hide yes)
@@
 			)
 		)
-		(property "Footprint" "BSPD:TSSOP-14_4.4x5mm_P0.65mm_TI_PW"
+		(property "Footprint" "TSSOP-14_4.4x5mm_P0.65mm_TI_PW"
 			(at 110.49 219.71 0)
 			(hide yes)
@@
 			)
 		)
-		(property "Footprint" "BSPD:TSSOP-14_4.4x5mm_P0.65mm_TI_PW"
+		(property "Footprint" "TSSOP-14_4.4x5mm_P0.65mm_TI_PW"
 			(at 111.76 90.17 0)
 			(hide yes)
@@
 			)
 		)
-		(property "Footprint" "BSPD:TSSOP-14_4.4x5mm_P0.65mm_TI_PW"
+		(property "Footprint" "TSSOP-14_4.4x5mm_P0.65mm_TI_PW"
 			(at 156.21 147.32 0)
 			(hide yes)
@@
 			)
 		)
-		(property "Footprint" "BSPD:TSSOP-14_4.4x5mm_P0.65mm_TI_PW"
+		(property "Footprint" "TSSOP-14_4.4x5mm_P0.65mm_TI_PW"
 			(at 99.06 120.65 0)
 			(hide yes)
@@
 			)
 		)
-		(property "Footprint" "BSPD:TSSOP-14_4.4x5mm_P0.65mm_TI_PW"
+		(property "Footprint" "TSSOP-14_4.4x5mm_P0.65mm_TI_PW"
 			(at 99.06 273.05 0)
 			(hide yes)
@@
 			)
 		)
-		(property "Footprint" "BSPD:TSSOP-14_4.4x5mm_P0.65mm_TI_PW"
+		(property "Footprint" "TSSOP-14_4.4x5mm_P0.65mm_TI_PW"
 			(at 97.79 250.19 0)
 			(hide yes)
@@
 			)
 		)
-		(property "Footprint" "BSPD:TSSOP-14_4.4x5mm_P0.65mm_TI_PW"
+		(property "Footprint" "TSSOP-14_4.4x5mm_P0.65mm_TI_PW"
 			(at 110.49 50.8 0)
 			(hide yes)
@@
 			)
 		)
-		(property "Footprint" "BSPD:TSSOP-14_4.4x5mm_P0.65mm_TI_PW"
+		(property "Footprint" "TSSOP-14_4.4x5mm_P0.65mm_TI_PW"
 			(at 100.33 143.51 0)
 			(hide yes)
@@
 			)
 		)
-		(property "Footprint" "BSPD:TSSOP-14_4.4x5mm_P0.65mm_TI_PW"
+		(property "Footprint" "TSSOP-14_4.4x5mm_P0.65mm_TI_PW"
 			(at 109.22 180.34 0)
 			(hide yes)

Commit message: autosave 2026-09-30 20:15:28
Parts:
- R1, R2, R3: footprint (none) -> Resistor_SMD:R_0805_2012Metric
Changed lines of the file:
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@@
 			)
 		)
-		(property "Footprint" ""
+		(property "Footprint" "Resistor_SMD:R_0805_2012Metric"
 			(at 299.72 35.56 0)
 			(hide yes)
@@
 			)
 		)
-		(property "Footprint" ""
+		(property "Footprint" "Resistor_SMD:R_0805_2012Metric"
 			(at 308.61 62.23 0)
 			(hide yes)
@@
 			)
 		)
-		(property "Footprint" ""
+		(property "Footprint" "Resistor_SMD:R_0805_2012Metric"
 			(at 299.72 57.15 0)
 			(hide yes)

Commit message: autosave 2026-09-30 20:17:37
Parts:
- C5: footprint Capacitor_SMD:C_1210_3225Metric -> Capacitor_SMD:C_0805_2012Metric
Changed lines of the file:
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@@
 			)
 		)
-		(property "Footprint" "Capacitor_SMD:C_1210_3225Metric"
+		(property "Footprint" "Capacitor_SMD:C_0805_2012Metric"
 			(at 139.7 22.86 0)
 			(hide yes)
