File: BSPD SAE.kicad_sch (KiCad schematic)
At the start: 37 parts, among them U1 LTC6994xS6-2, U3 TLV1824, U4 TLV1824

Commit message: autosave 2026-10-04 20:27:48
Other:
- note added: "Delay block"
- moved on the sheet: C11, C9, R1, R2, R3, R44, R45, R46, U1

Commit message: autosave 2026-10-04 21:16:58
Parts:
- added C10, C13: 10uf, Capacitor_SMD:C_0805_2012Metric, symbol Device:C_Small
- added C12: 100nf, Capacitor_SMD:C_0805_2012Metric, symbol Device:C_Small
- added R4: 102k, Resistor_SMD:R_0805_2012Metric, symbol Device:R_Small
- added R5: 309K, Resistor_SMD:R_0805_2012Metric, symbol Device:R_Small
- added U2: TPS7A2501DRVR, DRV0006A-IPC_A, symbol 2026-10-05_03-25-03:TPS7A2501DRVR
Connections:
- net 5V supply: now also C13.1, R5.1, U2.1 (OUT)
- net GND: now also C10.2, C12.2, C13.2, R4.2, U2.3 (PG), U2.5 (GND), U2.7 (Thermal_Pad)
- net Vsupply12: now also C10.1, C12.1, U2.4 (EN), U2.6 (IN)
- new net: R4.1, R5.2, U2.2 (FB)
Other:
- note added: "12v to 5v LDO linear regulator"
- moved on the sheet: C11, C9, R1, R2, R3, R44, R45, R46, U1

Commit message: autosave 2026-10-04 21:33:20
Parts:
- added D1: SS14, Diode_SMD:D_SMA, symbol Diode:SS14
Connections:
- net Vsupply12: now also D1.2 (A); no longer C10.1, C12.1, U2.4 (EN), U2.6 (IN)
- new net: C10.1, C12.1, D1.1 (K), U2.4 (EN), U2.6 (IN)
Other:
- moved on the sheet: C10
Changed lines of the file:
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@@
 	)
 	(junction
+		(at 245.11 97.79)
+		(diameter 0)
+		(color 0 0 0 0)
+	)
+	(junction
 		(at 110.49 250.19)
 		(diameter 0)
@@
 	)
 	(junction
-		(at 236.22 97.79)
-		(diameter 0)
-		(color 0 0 0 0)
-	)
-	(junction
 		(at 325.12 97.79)
 		(diameter 0)
@@
 	(wire
 		(pts
-			(xy 236.22 97.79) (xy 255.27 97.79)
+			(xy 74.93 118.11) (xy 87.63 118.11)
 		)
 		(stroke
@@
 	(wire
 		(pts
-			(xy 74.93 118.11) (xy 87.63 118.11)
+			(xy 46.99 184.15) (xy 101.6 184.15)
 		)
 		(stroke
@@
 	(wire
 		(pts
-			(xy 46.99 184.15) (xy 101.6 184.15)
+			(xy 269.24 107.95) (xy 269.24 97.79)
 		)
 		(stroke
@@
 	(wire
 		(pts
-			(xy 269.24 107.95) (xy 269.24 97.79)
+			(xy 307.34 113.03) (xy 316.23 113.03)
 		)
 		(stroke
@@
 	(wire
 		(pts
-			(xy 307.34 113.03) (xy 316.23 113.03)
+			(xy 269.24 46.99) (xy 269.24 52.07)
 		)
 		(stroke
@@
 	(wire
 		(pts
-			(xy 269.24 46.99) (xy 269.24 52.07)
+			(xy 278.13 30.48) (xy 288.29 30.48)
 		)
 		(stroke
@@
 	(wire
 		(pts
-			(xy 278.13 30.48) (xy 288.29 30.48)
+			(xy 82.55 215.9) (xy 97.79 215.9)
 		)
 		(stroke
@@
 	(wire
 		(pts
-			(xy 82.55 215.9) (xy 97.79 215.9)
+			(xy 245.11 97.79) (xy 255.27 97.79)
 		)
 		(stroke
@@
 	(wire
 		(pts
-			(xy 232.41 97.79) (xy 236.22 97.79)
+			(xy 232.41 97.79) (xy 234.95 97.79)
 		)
 		(stroke
@@
 	(wire
 		(pts
+			(xy 242.57 97.79) (xy 245.11 97.79)
+		)
+		(stroke
+			(width 0)
+			(type default)
+		)
+	)
+	(wire
+		(pts
 			(xy 128.27 40.64) (xy 128.27 50.8)
 		)
@@
 	)
 	(symbol
+		(lib_id "Diode:SS14")
+		(at 238.76 97.79 180)
+		(unit 1)
+		(body_style 1)
+		(exclude_from_sim no)
+		(in_bom yes)
+		(on_board yes)
+		(in_pos_files yes)
+		(dnp no)
+		(fields_autoplaced yes)
+		(property "Reference" "D1"
+			(at 239.0775 91.44 0)
+			(show_name no)
+			(do_not_autoplace no)
+			(effects
+				(font
+					(size 1.27 1.27)
+				)
+			)
+		)
+		(property "Value" "SS14"
+			(at 239.0775 93.98 0)
+			(show_name no)
+			(do_not_autoplace no)
+			(effects
+				(font
+					(size 1.27 1.27)
+				)
+			)
+		)
+		(property "Footprint" "Diode_SMD:D_SMA"
+			(at 238.76 93.345 0)
+			(hide yes)
+			(show_name no)
+			(do_not_autoplace no)
+			(effects
+				(font
+					(size 1.27 1.27)
+				)
+			)
+		)
+		(property "Datasheet" "https://www.vishay.com/docs/88746/ss12.pdf"
+			(at 238.76 97.79 0)
+			(hide yes)
+			(show_name no)
+			(do_not_autoplace no)
+			(effects
+				(font
+					(size 1.27 1.27)
+				)
+			)
+		)
+		(property "Description" "40V 1A Schottky Diode, SMA"
+			(at 238.76 97.79 0)
+			(hide yes)
+			(show_name no)
+			(do_not_autoplace no)
+			(effects
+				(font
+					(size 1.27 1.27)
+				)
+			)
+		)
+		(pin "2"
+		)
+		(pin "1"
+		)
+		(instances
+			(project "BSPD SAE"
+				(path "/136aa4d7-3b22-432f-9e98-3fb5ab08982d"
+					(reference "D1")
+					(unit 1)
+				)
+			)
+		)
+	)
+	(symbol
 		(lib_id "TLV1824:TLV1824")
 		(at 156.21 147.32 90)
@@
 	(symbol
 		(lib_id "power:GND")
-		(at 236.22 102.87 0)
+		(at 245.11 102.87 0)
 		(unit 1)
 		(body_style 1)
@@
 		(fields_autoplaced yes)
 		(property "Reference" "#PWR033"
-			(at 236.22 109.22 0)
+			(at 245.11 109.22 0)
 			(hide yes)
 			(show_name no)
@@
 		)
 		(property "Value" "GND"
-			(at 236.22 107.95 0)
+			(at 245.11 107.95 0)
 			(show_name no)
 			(do_not_autoplace no)
@@
 		)
 		(property "Footprint" ""
-			(at 236.22 102.87 0)
+			(at 245.11 102.87 0)
 			(hide yes)
 			(show_name no)
@@
 		)
 		(property "Datasheet" ""
-			(at 236.22 102.87 0)
+			(at 245.11 102.87 0)
 			(hide yes)
 			(show_name no)
@@
 		)
 		(property "Description" "Power symbol creates a global label with name \"GND\" , ground"
-			(at 236.22 102.87 0)
+			(at 245.11 102.87 0)
 			(hide yes)
 			(show_name no)
@@
 	(symbol
 		(lib_id "Device:C_Small")
-		(at 236.22 100.33 0)
+		(at 245.11 100.33 0)
 		(unit 1)
 		(body_style 1)
@@
 		(fields_autoplaced yes)
 		(property "Reference" "C10"
-			(at 238.76 99.0662 0)
+			(at 247.65 99.0662 0)
 			(show_name no)
 			(do_not_autoplace no)
@@
 		)
 		(property "Value" "10uf"
-			(at 238.76 101.6062 0)
+			(at 247.65 101.6062 0)
 			(show_name no)
 			(do_not_autoplace no)
@@
 		)
 		(property "Footprint" "Capacitor_SMD:C_0805_2012Metric"
-			(at 236.22 100.33 0)
+			(at 245.11 100.33 0)
 			(hide yes)
 			(show_name no)
@@
 		)
 		(property "Datasheet" "https://mm.digikey.com/Volume0/opasdata/d220001/medias/docus/962/UMK325C7106MM-T.pdf"
-			(at 236.22 100.33 0)
+			(at 245.11 100.33 0)
 			(hide yes)
 			(show_name no)
@@
 		)
 		(property "Description" "UMK325C7106MM-T Models"
-			(at 236.22 100.33 0)
+			(at 245.11 100.33 0)
 			(hide yes)
 			(show_name no)

Commit message: autosave 2026-10-04 22:53:10
Parts:
- added C14: 2.2uf, Capacitor_SMD:C_0805_2012Metric, symbol Device:C_Small
- added C15: 1uf, Capacitor_SMD:C_0805_2012Metric, symbol Device:C_Small
- added D2: BAT54C, Package_TO_SOT_SMD:SOT-23, symbol Diode:BAT54C
- added D3: 1N4148W, Diode_SMD:D_SOD-123, symbol Diode:1N4148W
- added Q1, Q3: MMBT3904, Package_TO_SOT_SMD:SOT-23, symbol Transistor_BJT:MMBT3904
- added Q2: 2N7002K, Package_TO_SOT_SMD:SOT-23, symbol Transistor_FET:2N7002K
- added R10: 100k, Resistor_SMD:R_0805_2012Metric, symbol Device:R_Small
- added R11: 1k, Resistor_SMD:R_0805_2012Metric, symbol Device:R_Small
- added R6: 4.7k, Resistor_SMD:R_0805_2012Metric, symbol Device:R_Small
- added R7: 47k, Resistor_SMD:R_0805_2012Metric, symbol Device:R_Small
- added R8: 1.5k, Resistor_SMD:R_0805_2012Metric, symbol Device:R_Small
- added R9: 22k, Resistor_SMD:R_0805_2012Metric, symbol Device:R_Small
Connections:
- net Brake_and_5KW_After_Delay: now also R8.1
- net GND: now also C15.2, D3.2 (A), Q1.2 (E), Q3.2 (E), R10.1, R11.1
- net Latch Input Sensor after 10ms: now also R7.2
- net Vsupply12: now also C14.1, R6.1
- new net: C15.1, D2.3, Q3.3 (C), R11.2
- new net: D2.1, Q1.3 (C), R6.2
- new net: D2.2, R8.2
- new net: Q1.1 (B), R7.1
- new net: C14.2, D3.1 (K), R10.2, R9.2
- new net: Q3.1 (B), R9.1
Other:
- note added: "12v to 5v LDO linear regulator data sheet : https://www.ti.com/lit/ds/symlink/tps7a25.pdf?HQS=dis-dk-null-digikeymode-dsf-pf-null-wwe&ts=1791170323719"
- note added: "Low When conditions arent met High when conditions are met->car turns off"
- note added: "Reads High when everything is reading good Reads Low when/ if faults in sensors"
- note added: "data sheet: https://www.ti.com/lit/ds/symlink/tlv1824-q1.pdf?ts=1791174079110&ref_url=https%253A%252F%252Fwww.ti.com%252Fproduct%252FTLV1824-Q1"
- note removed: "12v to 5v LDO linear regulator"

Commit message: autosave 2026-10-04 23:07:30
Parts:
- added CR1: MCR100-8, SOT23_DIO, symbol 2026-10-05_05-48-00:MCR100-8
- added R12, R13, R14, R15: 1k, Resistor_SMD:R_0805_2012Metric, symbol Device:R_Small
- R7: value 47k -> 22k
Connections:
- net GND: now also Q2.2 (S), CR1.2, R13.1
- net Vsupply12: now also R14.1, R15.1
- net at C15.1, D2.3, Q3.3 (C)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: now also CR1.1
- net at Q2.1 (G): now also R12.1, R13.2
- new net: CR1.3, R12.2, R14.2, R15.2
Other:
- moved on the sheet: Q2

Commit message: autosave 2026-10-05 00:11:05
Parts:
- added D4: SS14, Diode_SMD:D_SMA, symbol Diode:SS14
- added J1: 430450412, CONN_SD-43045-005_04_MOL, symbol 2026-10-05_06-33-49:430450412
- added J2: 436500215, CONN_SD-43650-006_02_MOL, symbol 2026-10-05_06-36-43:436500215
- added K1: G5Q-1A-EU DC12, RELAY_G5Q-1A DC5_OMR, symbol 2026-10-05_06-05-09:G5Q-1A-EU_DC12
- R12, R13: value 1k -> 10k
Connections:
- net 5kw level: now also J1.3
- net Brake Sensor: now also J1.4
- net GND: now also J1.2
- net Vsupply12: now also D4.1 (K), J1.1, K1.1
- net at Q2.3 (D): now also D4.2 (A), K1.5
- new net SDC_IN: J2.1, K1.2
- new net SDC_OUT: J2.2, K1.3
Other:
- note added: "Connectors"
- note added: "Latching Circuit"
- moved on the sheet: C14, C15, CR1, D2, D3, Q1, Q2, Q3, R10, R11, R12, R13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

Commit message: autosave 2026-10-07 12:15:04
Other:
- note added: "Comparator used :TLV1824 Logic explained: U3A is in charge of checking whether or not 5KW demand condition is being met by the motor by comparing voltage from a IC to a fixed voltge. U3B is comparing whether or not there is an issue in the wire or sensor. It does this by checking if a voltage higher than .5V is being recieved. Goes High when More than .5 is being read by the comparator and low Wh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"
- note removed: "Comparator used :TLV1824 Logic explained U3A is what will be used to compare the actual signal level with U4A. If U3A outputs high that means we have reached 5KW demand Per Rule book limits While U3B and U3C are wired the opposite way both will output high if there conditions arent met. when they pull low this indicates a problem with the wiring which will shutdown the car instantly"
Changed lines of the file:
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@@
 		)
 	)
-	(text "Comparator used :TLV1824\nLogic explained U3A is what will be used to compare the actual signal\nlevel with U4A. If U3A outputs high that means we have reached 5KW demand \nPer Rule book limits\n\nWhile U3B and U3C are wired the opposite way both will output high if\nthere conditions arent met. when they pull low this indicates a problem\nwith the wiring which will shutdown the car instantly\n"
+	(text "Comparator used :TLV1824\nLogic explained: U3A is in charge of checking whether or not 5KW demand condition\nis being met by the motor by comparing voltage from a IC to a fixed voltge.\n\nU3B is comparing whether or not there is an issue in the wire or sensor. It does \nthis by checking if a voltage higher than .5V is being recieved. Goes High when \nMore than .5 is being read by the comparator and low When less then 5 is being Read.\n\nU3C checks wether there is a short or issue with the output of the sensor which would leed\nto more than 4.5V being sent to the BSPD. IT sits high when no fault is being detected by the \ncomparator and falls low when more than 4.5v is being sent to the comparator."
 		(exclude_from_sim no)
 		(at -46.228 64.008 0)

Commit message: autosave 2026-10-14 10:46:15
Parts:
- removed J1: 430450412, CONN_SD-43045-005_04_MOL, symbol 2026-10-05_06-33-49:430450412
- removed J2: 436500215, CONN_SD-43650-006_02_MOL, symbol 2026-10-05_06-36-43:436500215
- added J3: DT13-6P, TE_DT13-6P, symbol DT13-6P:DT13-6P
- R18, R19, R23, R28, R29, R34, R35, R36, R37, R38, R44, R45, R46: PROD_ID RMCF0805FT10K0 -> RES-07856
- R20, R24, R30, R39, R40, R42: PROD_ID RG2012P-105-B-T5 -> RES-07856
Connections:
- net 5kw level: now also J3.3
- net Brake Sensor: now also J3.4
- net GND: now also J3.2
- net SDC_IN: now also J3.5
- net SDC_OUT: now also J3.6
- net Vsupply12: now also J3.1
