File: BSPD SAE.kicad_sch (KiCad schematic)
At the start: 74 parts, among them J2 436500215, J3 430450612, K1 G5Q-1A-EU DC12, Q1 MMBT3904, Q2 2N7002K, Q3 MMBT3904, U1 LTC6994xS6-2, U2 TPS7A2501DRVR, U3 TLV1824, U4 TLV1824

Commit message: autosave 2026-10-26 22:13:31
Parts:
- added R21, R25, R31, R41, R43, R47, R48, R49, R50, R51, R52, R53: 10k, Resistor_SMD:R_0805_2012Metric, symbol PCM_SparkFun-Resistor:R_Small
Connections:
- net 5V supply: now also R21.1, R31.1, R43.1, R48.2, R50.2, R52.2; no longer R17.1, R22.1, R26.1, R27.1, R32.1, R33.1
- net GND: now also R25.2, R41.2, R47.1, R49.1, R51.1, R53.1; no longer R17.3, R22.3, R26.3, R27.3, R32.3, R33.3
- new net: R22.1, R31.2
- new net: R26.1, R48.1
- new net: R22.3, R41.1
- new net: R33.1, R50.1
- new net: R26.3, R49.2
- new net: R17.1, R21.2
- new net: R33.3, R51.2
- new net: R17.3, R25.1
- new net: R32.1, R52.1
- new net: R27.3, R47.2
- new net: R27.1, R43.2
- new net: R32.3, R53.2
Other:
- moved on the sheet: C7, C8, R22, R23, R24, R26, R27, R28, R29, R30, R32, R33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

Commit message: autosave 2026-10-28 01:28:09
Parts:
- R21, R31, R43, R48, R50, R52: value 10k -> 309k
- R25, R41, R47, R49, R51, R53: value 10k -> 20k
Changed lines of the file:
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@@
 			)
 		)
-		(property "Value" "10k"
+		(property "Value" "309k"
 			(at 34.29 93.98 0)
 			(show_name no)
@@
 			)
 		)
-		(property "Value" "10k"
+		(property "Value" "309k"
 			(at 41.91 226.0599 90)
 			(show_name no)
@@
 			)
 		)
-		(property "Value" "10k"
+		(property "Value" "309k"
 			(at 64.77 281.9399 90)
 			(show_name no)
@@
 			)
 		)
-		(property "Value" "10k"
+		(property "Value" "20k"
 			(at 34.29 121.92 0)
 			(show_name no)
@@
 			)
 		)
-		(property "Value" "10k"
+		(property "Value" "309k"
 			(at 36.83 40.64 0)
 			(show_name no)
@@
 			)
 		)
-		(property "Value" "10k"
+		(property "Value" "20k"
 			(at 64.77 314.9599 90)
 			(show_name no)
@@
 			)
 		)
-		(property "Value" "10k"
+		(property "Value" "309k"
 			(at 49.53 345.4399 90)
 			(show_name no)
@@
 			)
 		)
-		(property "Value" "10k"
+		(property "Value" "20k"
 			(at 36.83 68.58 0)
 			(show_name no)
@@
 			)
 		)
-		(property "Value" "10k"
+		(property "Value" "20k"
 			(at 40.64 190.4999 90)
 			(show_name no)
@@
 			)
 		)
-		(property "Value" "10k"
+		(property "Value" "20k"
 			(at 49.53 374.6499 90)
 			(show_name no)
@@
 			)
 		)
-		(property "Value" "10k"
+		(property "Value" "20k"
 			(at 41.91 264.1599 90)
 			(show_name no)
@@
 			)
 		)
-		(property "Value" "10k"
+		(property "Value" "309k"
 			(at 34.29 157.48 0)
 			(show_name no)

Commit message: autosave 2026-10-28 02:00:57
Parts:
- R21: value 309k -> 200k
- R25: value 20k -> 8.25k
- R43, R52: value 309k -> 5k
- R47, R53: value 20k -> 110k
- R48: value 309k -> place holder
- R49: value 20k -> place holder
Changed lines of the file:
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@@
 			)
 		)
-		(property "Value" "309k"
+		(property "Value" "place holder"
 			(at 41.91 226.0599 90)
 			(show_name no)
@@
 			)
 		)
-		(property "Value" "309k"
+		(property "Value" "200k"
 			(at 36.83 40.64 0)
 			(show_name no)
@@
 			)
 		)
-		(property "Value" "309k"
+		(property "Value" "5k"
 			(at 49.53 345.4399 90)
 			(show_name no)
@@
 			)
 		)
-		(property "Value" "20k"
+		(property "Value" "8.25k"
 			(at 36.83 68.58 0)
 			(show_name no)
@@
 			)
 		)
-		(property "Value" "20k"
+		(property "Value" "110k"
 			(at 40.64 190.4999 90)
 			(show_name no)
@@
 			)
 		)
-		(property "Value" "20k"
+		(property "Value" "110k"
 			(at 49.53 374.6499 90)
 			(show_name no)
@@
 			)
 		)
-		(property "Value" "20k"
+		(property "Value" "place holder"
 			(at 41.91 264.1599 90)
 			(show_name no)
@@
 			)
 		)
-		(property "Value" "309k"
+		(property "Value" "5k"
 			(at 34.29 157.48 0)
 			(show_name no)

Commit message: autosave 2026-10-28 02:07:07
Parts:
- R21: value 200k -> 76.8k
- R25: value 8.25k -> 84.5k
Changed lines of the file:
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@@
 			)
 		)
-		(property "Value" "200k"
+		(property "Value" "76.8k"
 			(at 36.83 40.64 0)
 			(show_name no)
@@
 			)
 		)
-		(property "Value" "8.25k"
+		(property "Value" "84.5k"
 			(at 36.83 68.58 0)
 			(show_name no)

Commit message: autosave 2026-10-28 02:11:13
Parts:
- added C16, C17: 100nf, Capacitor_SMD:C_0805_2012Metric, symbol Device:C_Small
Connections:
- net GND: now also C16.1, C17.1
- net at R18.1, R20.1, U3.5 (+): now also C16.2
- net at R37.2, R42.1, U4.5 (+): now also C17.2

Commit message: autosave 2026-10-28 02:15:19
Parts:
- removed C16, C17: 100nf, Capacitor_SMD:C_0805_2012Metric, symbol Device:C_Small
- R43, R52: value 5k -> 4.99k

Commit message: autosave 2026-10-28 02:21:28
Parts:
- R1: value 1M -> 523k
- R2: value 523k -> 1000k
Changed lines of the file:
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@@
 			)
 		)
-		(property "Value" "1M"
+		(property "Value" "523k"
 			(at 271.78 34.2899 0)
 			(show_name no)
@@
 			)
 		)
-		(property "Value" "523k"
+		(property "Value" "1000k"
 			(at 271.78 55.8799 0)
 			(show_name no)

Commit message: autosave 2026-10-28 02:31:43
Parts:
- removed C15: 1uf, Capacitor_SMD:C_0805_2012Metric, symbol Device:C_Small
- removed CR1: MCR100-8, SOT23_DIO, symbol 2026-10-05_05-48-00:MCR100-8
- removed Q1: MMBT3904, Package_TO_SOT_SMD:SOT-23, symbol Transistor_BJT:MMBT3904
- removed R11, R14, R15: 1k, Resistor_SMD:R_0805_2012Metric, symbol Device:R_Small
- removed R6: 4.7k, Resistor_SMD:R_0805_2012Metric, symbol Device:R_Small
- removed R7: 22k, Resistor_SMD:R_0805_2012Metric, symbol Device:R_Small
