File: BSPD SAE.kicad_pcb (KiCad board)
At the start: 2 copper layers, 30 parts

Commit message: autosave 2026-09-30 20:15:28
Parts:
- added C11: 100nf, Capacitor_SMD:C_0805_2012Metric, F.Cu at (105.7, 85.1)
- added U1: LTC6994xS6-2, Package_TO_SOT_SMD:TSOT-23-6, F.Cu at (106.1, 81.4)
- added U3: TLV1824, MYLIB:TSSOP-14_4.4x5mm_P0.65mm_TI_PW, F.Cu at (96.9, 83.8)
- added U4: TLV1824, MYLIB:TSSOP-14_4.4x5mm_P0.65mm_TI_PW, F.Cu at (96.9, 90.5)

Commit message: autosave 2026-09-30 20:17:37
Parts:
- added R1: 1M, Resistor_SMD:R_0805_2012Metric, F.Cu at (99.2, 68.5)
- added R2: 523k, Resistor_SMD:R_0805_2012Metric, F.Cu at (99.2, 71.4)
- added R3: 715K, Resistor_SMD:R_0805_2012Metric, F.Cu at (99.2, 74.4)
- C5: footprint Capacitor_SMD:C_1210_3225Metric -> Capacitor_SMD:C_0805_2012Metric
- moved C5 6.13 mm to (88.0, 83.0)

Commit message: autosave 2026-10-04 21:31:17
Parts:
- added C10: 10uf, Capacitor_SMD:C_0805_2012Metric, F.Cu at (115.5, 74.2)
- added C12: 100nf, Capacitor_SMD:C_0805_2012Metric, F.Cu at (115.5, 77.2)
- added C13: 10uf, Capacitor_SMD:C_0805_2012Metric, F.Cu at (115.5, 80.2)
- added R4: 102k, Resistor_SMD:R_0805_2012Metric, F.Cu at (119.9, 74.1)
- added R5: 309K, Resistor_SMD:R_0805_2012Metric, F.Cu at (119.9, 77.1)
- added U2: TPS7A2501DRVR, MYLIB:DRV0006A-IPC_A, F.Cu at (115.8, 91.9)

Commit message: autosave 2026-10-05 00:02:50
Parts:
- added C14: 2.2uf, Capacitor_SMD:C_0805_2012Metric, F.Cu at (152.6, 58.9)
- added C15: 1uf, Capacitor_SMD:C_0805_2012Metric, F.Cu at (152.6, 61.9)
- added CR1: MCR100-8, MYLIB:SOT23_DIO, F.Cu at (153.9, 65.9)
- added D1: SS14, Diode_SMD:D_SMA, F.Cu at (129.0, 81.3)
- added D2: BAT54C, Package_TO_SOT_SMD:SOT-23, F.Cu at (139.1, 59.6)
- added D3: 1N4148W, Diode_SMD:D_SOD-123, F.Cu at (153.3, 70.1)
- added D4: SS14, Diode_SMD:D_SMA, F.Cu at (129.0, 85.9)
- added J1: 430450412, MYLIB:CONN_SD-43045-005_04_MOL, F.Cu at (149.0, 86.7)
- added J2: 436500215, MYLIB:CONN_SD-43650-006_02_MOL, F.Cu at (149.0, 76.1)
- added K1: G5Q-1A-EU DC12, MYLIB:RELAY_G5Q-1A DC5_OMR, F.Cu at (134.6, 77.1)
- added Q1: MMBT3904, Package_TO_SOT_SMD:SOT-23, F.Cu at (139.1, 64.1)
- added Q2: 2N7002K, Package_TO_SOT_SMD:SOT-23, F.Cu at (139.1, 68.5)
- added Q3: MMBT3904, Package_TO_SOT_SMD:SOT-23, F.Cu at (139.1, 73.0)
- added R10: 100k, Resistor_SMD:R_0805_2012Metric, F.Cu at (143.8, 70.7)
- added R11: 1k, Resistor_SMD:R_0805_2012Metric, F.Cu at (148.2, 58.9)
- added R12: 10k, Resistor_SMD:R_0805_2012Metric, F.Cu at (148.2, 61.8)
- added R13: 10k, Resistor_SMD:R_0805_2012Metric, F.Cu at (148.2, 64.8)
- added R14: 1k, Resistor_SMD:R_0805_2012Metric, F.Cu at (148.2, 67.7)
- added R15: 1k, Resistor_SMD:R_0805_2012Metric, F.Cu at (148.2, 70.7)
- added R6: 4.7k, Resistor_SMD:R_0805_2012Metric, F.Cu at (143.8, 58.9)
- added R7: 22k, Resistor_SMD:R_0805_2012Metric, F.Cu at (143.8, 61.8)
- added R8: 1.5k, Resistor_SMD:R_0805_2012Metric, F.Cu at (143.8, 64.8)
- added R9: 22k, Resistor_SMD:R_0805_2012Metric, F.Cu at (143.8, 67.7)
Connections:
- C10 pad 1: Vsupply12 -> Net-(D1-K)
- C12 pad 1: Vsupply12 -> Net-(D1-K)
- U2 pad 4: Vsupply12 -> Net-(D1-K)
- U2 pad 6: Vsupply12 -> Net-(D1-K)
