File: BSPD SAE.kicad_pcb (KiCad board)
At the start: 2 copper layers, 66 parts, among them J1 430450412, J2 436500215, K1 G5Q-1A-EU DC12, Q1 MMBT3904, Q2 2N7002K, Q3 MMBT3904, U1 LTC6994xS6-2, U2 TPS7A2501DRVR, U3 TLV1824, U4 TLV1824

Commit message: autosave 2026-10-06 17:10:39
Parts:
- moved C13 67.3 mm to (167.4, 123.0), turned to 90 degrees
- moved R5 64.3 mm to (164.9, 123.0), turned to 90 degrees
- moved R4 63.3 mm to (164.9, 118.7), turned to 180 degrees
- moved R32 60.4 mm to (125.0, 120.0), turned to 90 degrees
- moved C12 60.4 mm to (156.9, 121.2), turned to 180 degrees
- moved C10 60.1 mm to (156.9, 117.7), turned to 180 degrees
- moved R26 58.1 mm to (125.0, 99.0), turned to 90 degrees
- moved U3 56.0 mm to (143.9, 72.0)
- moved C14 55.1 mm to (106.5, 28.6)
- moved C15 55.1 mm to (106.5, 31.6)
- moved CR1 55.1 mm to (107.8, 35.6)
- moved D2 55.1 mm to (93.0, 29.3)
- moved D3 55.1 mm to (107.2, 39.8)
- moved Q1 55.1 mm to (93.0, 33.7)
- moved Q2 55.1 mm to (93.0, 38.2)
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Other:
- board outline added: 70 x 70 mm

Commit message: autosave 2026-10-06 17:12:47
Parts:
- moved C7 6.52 mm to (137.0, 97.0)
- moved C8 6.52 mm to (139.0, 97.0)
- moved U4 6.52 mm to (147.5, 97.0)
- moved C10 6.08 mm to (150.9, 116.7)
- moved C12 6.08 mm to (150.9, 120.2)
- moved C13 6.08 mm to (161.4, 122.1)
- moved D1 6.08 mm to (148.0, 112.5)
- moved J1 6.08 mm to (140.5, 117.5)
- moved R4 6.08 mm to (158.9, 117.7)
- moved R5 6.08 mm to (158.9, 122.1)
- moved U2 6.08 mm to (155.4, 120.2)
- moved C5 5.88 mm to (136.6, 77.0)
- moved C6 5.88 mm to (138.6, 77.0)
- moved U3 5.88 mm to (147.0, 77.0)
Changed lines of the file:
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@@
 	(footprint "Capacitor_SMD:C_0805_2012Metric"
 		(layer "F.Cu")
-		(at 156.871968 121.150001 180)
+		(at 150.871968 120.150002 180)
 		(descr "Capacitor SMD 0805 (2012 Metric), square (rectangular) end terminal, IPC-7351 nominal, (Body size source: IPC-SM-782 page 76, https://www.pcb-3d.com/wordpress/wp-content/uploads/ipc-sm-782a_amendment_1_and_2.pdf, https://docs.google.com/spreadsheets/d/1BsfQQcO9C6DZCsRaXUlFlo91Tg2WpOkGARC1WS5S8t0/edit?usp=sharing)")
 		(tags "capacitor")
@@
 	(footprint "MYLIB:CONN_SD-43045-005_04_MOL"
 		(layer "F.Cu")
-		(at 146.499999 118.5 90)
+		(at 140.499999 117.500001 90)
 		(tags "430450412 ")
 		(property "Reference" "J1"
@@
 	(footprint "Resistor_SMD:R_0805_2012Metric"
 		(layer "F.Cu")
-		(at 164.921968 123.05 90)
+		(at 158.921968 122.050001 90)
 		(descr "Resistor SMD 0805 (2012 Metric), square (rectangular) end terminal, IPC-7351 nominal, (Body size source: IPC-SM-782 page 72, https://www.pcb-3d.com/wordpress/wp-content/uploads/ipc-sm-782a_amendment_1_and_2.pdf)")
 		(tags "resistor")
@@
 	(footprint "MYLIB:TSSOP-14_4.4x5mm_P0.65mm_TI_PW"
 		(layer "F.Cu")
-		(at 143.9 72)
+		(at 147 77)
 		(descr "TI PW (R-PDSO-G14) TSSOP-14, 4.4x5.0mm body, 0.65mm pitch, for TLV1824PWR, land pattern per TI PW0014A (datasheet SNOSDC8E p.52)")
 		(tags "TSSOP 14 0.65 PW TI TLV1824")
@@
 	(footprint "Capacitor_SMD:C_0805_2012Metric"
 		(layer "F.Cu")
-		(at 133.5 102.55 -90)
+		(at 137 97.05 -90)
 		(descr "Capacitor SMD 0805 (2012 Metric), square (rectangular) end terminal, IPC-7351 nominal, (Body size source: IPC-SM-782 page 76, https://www.pcb-3d.com/wordpress/wp-content/uploads/ipc-sm-782a_amendment_1_and_2.pdf, https://docs.google.com/spreadsheets/d/1BsfQQcO9C6DZCsRaXUlFlo91Tg2WpOkGARC1WS5S8t0/edit?usp=sharing)")
 		(tags "capacitor")
@@
 	(footprint "Capacitor_SMD:C_0805_2012Metric"
 		(layer "F.Cu")
-		(at 135.5 102.5 -90)
+		(at 139 97 -90)
 		(descr "Capacitor SMD 0805 (2012 Metric), square (rectangular) end terminal, IPC-7351 nominal, (Body size source: IPC-SM-782 page 76, https://www.pcb-3d.com/wordpress/wp-content/uploads/ipc-sm-782a_amendment_1_and_2.pdf, https://docs.google.com/spreadsheets/d/1BsfQQcO9C6DZCsRaXUlFlo91Tg2WpOkGARC1WS5S8t0/edit?usp=sharing)")
 		(tags "capacitor")
@@
 	(footprint "Capacitor_SMD:C_0805_2012Metric"
 		(layer "F.Cu")
-		(at 156.921968 117.650001 180)
+		(at 150.921968 116.650002 180)
 		(descr "Capacitor SMD 0805 (2012 Metric), square (rectangular) end terminal, IPC-7351 nominal, (Body size source: IPC-SM-782 page 76, https://www.pcb-3d.com/wordpress/wp-content/uploads/ipc-sm-782a_amendment_1_and_2.pdf, https://docs.google.com/spreadsheets/d/1BsfQQcO9C6DZCsRaXUlFlo91Tg2WpOkGARC1WS5S8t0/edit?usp=sharing)")
 		(tags "capacitor")
@@
 	(footprint "Capacitor_SMD:C_0805_2012Metric"
 		(layer "F.Cu")
-		(at 133.5 72.05 -90)
+		(at 136.6 77.05 -90)
 		(descr "Capacitor SMD 0805 (2012 Metric), square (rectangular) end terminal, IPC-7351 nominal, (Body size source: IPC-SM-782 page 76, https://www.pcb-3d.com/wordpress/wp-content/uploads/ipc-sm-782a_amendment_1_and_2.pdf, https://docs.google.com/spreadsheets/d/1BsfQQcO9C6DZCsRaXUlFlo91Tg2WpOkGARC1WS5S8t0/edit?usp=sharing)")
 		(tags "capacitor")
@@
 	(footprint "Diode_SMD:D_SMA"
 		(layer "F.Cu")
-		(at 154 113.5 180)
+		(at 148 112.500001 180)
 		(descr "Diode SMA (DO-214AC)")
 		(tags "Diode SMA (DO-214AC)")
@@
 	(footprint "Resistor_SMD:R_0805_2012Metric"
 		(layer "F.Cu")
-		(at 164.921968 118.650001 180)
+		(at 158.921968 117.650002 180)
 		(descr "Resistor SMD 0805 (2012 Metric), square (rectangular) end terminal, IPC-7351 nominal, (Body size source: IPC-SM-782 page 72, https://www.pcb-3d.com/wordpress/wp-content/uploads/ipc-sm-782a_amendment_1_and_2.pdf)")
 		(tags "resistor")
@@
 	(footprint "MYLIB:TSSOP-14_4.4x5mm_P0.65mm_TI_PW"
 		(layer "F.Cu")
-		(at 144 102.5)
+		(at 147.5 97)
 		(descr "TI PW (R-PDSO-G14) TSSOP-14, 4.4x5.0mm body, 0.65mm pitch, for TLV1824PWR, land pattern per TI PW0014A (datasheet SNOSDC8E p.52)")
 		(tags "TSSOP 14 0.65 PW TI TLV1824")
@@
 	(footprint "Capacitor_SMD:C_0805_2012Metric"
 		(layer "F.Cu")
-		(at 135.5 72.05 -90)
+		(at 138.6 77.05 -90)
 		(descr "Capacitor SMD 0805 (2012 Metric), square (rectangular) end terminal, IPC-7351 nominal, (Body size source: IPC-SM-782 page 76, https://www.pcb-3d.com/wordpress/wp-content/uploads/ipc-sm-782a_amendment_1_and_2.pdf, https://docs.google.com/spreadsheets/d/1BsfQQcO9C6DZCsRaXUlFlo91Tg2WpOkGARC1WS5S8t0/edit?usp=sharing)")
 		(tags "capacitor")
@@
 	(footprint "MYLIB:DRV0006A-IPC_A"
 		(layer "F.Cu")
-		(at 161.421968 121.150001 180)
+		(at 155.421968 120.150002 180)
 		(tags "TPS7A2501DRVR ")
 		(property "Reference" "U2"
@@
 	(footprint "Capacitor_SMD:C_0805_2012Metric"
 		(layer "F.Cu")
-		(at 167.421968 123.05 90)
+		(at 161.421968 122.050001 90)
 		(descr "Capacitor SMD 0805 (2012 Metric), square (rectangular) end terminal, IPC-7351 nominal, (Body size source: IPC-SM-782 page 76, https://www.pcb-3d.com/wordpress/wp-content/uploads/ipc-sm-782a_amendment_1_and_2.pdf, https://docs.google.com/spreadsheets/d/1BsfQQcO9C6DZCsRaXUlFlo91Tg2WpOkGARC1WS5S8t0/edit?usp=sharing)")
 		(tags "capacitor")

Commit message: autosave 2026-10-06 17:27:29
Parts:
- moved U1 105.7 mm to (158.9, 88.5)
- moved C12 4.68 mm to (146.4, 121.7)
- moved C13 4.68 mm to (157.0, 123.6)
- moved R5 4.68 mm to (154.5, 123.6)
- moved C10 4.68 mm to (146.5, 118.2)
- moved R4 4.68 mm to (154.5, 119.2)
- moved U2 4.68 mm to (151.0, 121.7)
- moved D1 1.12 mm to (147.5, 113.5)
Changed lines of the file:
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@@
 	(footprint "Capacitor_SMD:C_0805_2012Metric"
 		(layer "F.Cu")
-		(at 150.871968 120.150002 180)
+		(at 146.45 121.687501 180)
 		(descr "Capacitor SMD 0805 (2012 Metric), square (rectangular) end terminal, IPC-7351 nominal, (Body size source: IPC-SM-782 page 76, https://www.pcb-3d.com/wordpress/wp-content/uploads/ipc-sm-782a_amendment_1_and_2.pdf, https://docs.google.com/spreadsheets/d/1BsfQQcO9C6DZCsRaXUlFlo91Tg2WpOkGARC1WS5S8t0/edit?usp=sharing)")
 		(tags "capacitor")
@@
 	(footprint "Resistor_SMD:R_0805_2012Metric"
 		(layer "F.Cu")
-		(at 158.921968 122.050001 90)
+		(at 154.5 123.5875 90)
 		(descr "Resistor SMD 0805 (2012 Metric), square (rectangular) end terminal, IPC-7351 nominal, (Body size source: IPC-SM-782 page 72, https://www.pcb-3d.com/wordpress/wp-content/uploads/ipc-sm-782a_amendment_1_and_2.pdf)")
 		(tags "resistor")
@@
 	(footprint "Capacitor_SMD:C_0805_2012Metric"
 		(layer "F.Cu")
-		(at 150.921968 116.650002 180)
+		(at 146.5 118.187501 180)
 		(descr "Capacitor SMD 0805 (2012 Metric), square (rectangular) end terminal, IPC-7351 nominal, (Body size source: IPC-SM-782 page 76, https://www.pcb-3d.com/wordpress/wp-content/uploads/ipc-sm-782a_amendment_1_and_2.pdf, https://docs.google.com/spreadsheets/d/1BsfQQcO9C6DZCsRaXUlFlo91Tg2WpOkGARC1WS5S8t0/edit?usp=sharing)")
 		(tags "capacitor")
@@
 	(footprint "Diode_SMD:D_SMA"
 		(layer "F.Cu")
-		(at 148 112.500001 180)
+		(at 147.5 113.5 180)
 		(descr "Diode SMA (DO-214AC)")
 		(tags "Diode SMA (DO-214AC)")
@@
 	(footprint "Resistor_SMD:R_0805_2012Metric"
 		(layer "F.Cu")
-		(at 158.921968 117.650002 180)
+		(at 154.5 119.187501 180)
 		(descr "Resistor SMD 0805 (2012 Metric), square (rectangular) end terminal, IPC-7351 nominal, (Body size source: IPC-SM-782 page 72, https://www.pcb-3d.com/wordpress/wp-content/uploads/ipc-sm-782a_amendment_1_and_2.pdf)")
 		(tags "resistor")
@@
 	(footprint "Package_TO_SOT_SMD:TSOT-23-6"
 		(layer "F.Cu")
-		(at 60.029 51.053)
+		(at 158.8625 88.45)
 		(descr "TSOT, 6 Pin (https://www.jedec.org/sites/default/files/docs/MO-193D.pdf variant AA)")
 		(tags "TSOT TO_SOT_SMD")
@@
 	(footprint "MYLIB:DRV0006A-IPC_A"
 		(layer "F.Cu")
-		(at 155.421968 120.150002 180)
+		(at 151 121.687501 180)
 		(tags "TPS7A2501DRVR ")
 		(property "Reference" "U2"
@@
 	(footprint "Capacitor_SMD:C_0805_2012Metric"
 		(layer "F.Cu")
-		(at 161.421968 122.050001 90)
+		(at 157 123.5875 90)
 		(descr "Capacitor SMD 0805 (2012 Metric), square (rectangular) end terminal, IPC-7351 nominal, (Body size source: IPC-SM-782 page 76, https://www.pcb-3d.com/wordpress/wp-content/uploads/ipc-sm-782a_amendment_1_and_2.pdf, https://docs.google.com/spreadsheets/d/1BsfQQcO9C6DZCsRaXUlFlo91Tg2WpOkGARC1WS5S8t0/edit?usp=sharing)")
 		(tags "capacitor")

Commit message: autosave 2026-10-13 16:31:22
Parts:
- moved R35 129.7 mm to (153.0, 98.6), turned to 90 degrees
- moved R36 129.0 mm to (156.0, 94.4), turned to 90 degrees
- moved R34 128.6 mm to (135.0, 118.5), turned to 90 degrees
- moved R19 128.0 mm to (135.0, 112.5), turned to 90 degrees
- moved R29 122.8 mm to (156.0, 71.6), turned to 90 degrees
- moved R39 122.6 mm to (153.0, 94.5), turned to 90 degrees
- moved R28 121.8 mm to (153.0, 76.5), turned to 90 degrees
- moved R30 120.6 mm to (153.0, 71.5), turned to 90 degrees
- moved R38 113.0 mm to (138.0, 100.0), turned to 90 degrees
- moved R37 111.5 mm to (134.5, 100.0), turned to -90 degrees
- moved R40 109.8 mm to (132.5, 94.5), turned to 90 degrees
- moved R42 109.7 mm to (134.5, 94.5), turned to 90 degrees
- moved R18 108.3 mm to (133.0, 76.5), turned to 90 degrees
- moved R23 108.0 mm to (136.5, 76.5), turned to 90 degrees
- moved R1 103.6 mm to (145.1, 86.0)
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
Commit message: autosave 2026-10-13 17:18:04
Parts:
- moved Q2 83.2 mm to (171.4, 64.5), turned to 90 degrees
- moved D4 83.1 mm to (175.9, 62.5), turned to 90 degrees
- moved Q3 79.7 mm to (174.0, 82.5), turned to 180 degrees
- moved R9 72.2 mm to (174.0, 87.0)
- moved R13 72.1 mm to (172.9, 70.0), turned to 90 degrees
- moved R10 69.4 mm to (170.5, 87.9), turned to 90 degrees
- moved D2 68.4 mm to (165.3, 78.9)
- moved R14 68.3 mm to (166.8, 70.0), turned to -90 degrees
- moved R12 68.1 mm to (169.9, 70.0), turned to 90 degrees
- moved R15 67.4 mm to (163.9, 70.0), turned to -90 degrees
- moved C9 64.6 mm to (151.5, 81.0), turned to 90 degrees
- moved Q1 63.7 mm to (159.0, 79.0), turned to 90 degrees
- moved R8 63.6 mm to (161.5, 75.0), turned to -90 degrees
- moved CR1 61.9 mm to (169.9, 76.5)
- moved R11 61.5 mm to (168.4, 82.5), turned to 90 degrees
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
Commit message: autosave 2026-10-15 17:01:41
Routing:
- net GND: track 0.00 -> 10.5 mm, vias 0 -> 24
- added copper zone on In1.Cu, net GND
Other:
- copper layers 2 -> 4

Commit message: autosave 2026-10-15 17:32:55
Parts:
- moved R32 12.1 mm to (131.0, 109.5)
- moved C13 8.96 mm to (168.0, 104.0)
- moved R5 8.96 mm to (165.5, 104.0)
- moved C10 8.54 mm to (157.5, 99.7)
- moved C12 8.54 mm to (157.5, 103.2)
- moved D1 8.54 mm to (158.5, 95.0)
- moved J1 8.54 mm to (151.5, 99.0)
- moved R19 8.54 mm to (143.0, 96.5)
- moved R34 8.54 mm to (143.0, 102.5)
- moved R4 8.54 mm to (165.5, 100.7)
- moved U2 8.54 mm to (162.0, 103.2)
Routing:
- net GND: track 10.5 -> 40.7 mm, vias 24 -> 29
- net 5V supply: track 0.00 -> 12.5 mm, vias 0 -> 7
- added copper zone on In2.Cu, net 5V supply
Other:
- board size 70 x 70 mm -> 70 x 69 mm
