File: BSPD SAE.kicad_pcb (KiCad board)
At the start: 4 copper layers, 70 x 50.3 mm, 74 parts, among them J1 430450412, J2 436500215, K1 G5Q-1A-EU DC12, Q1 MMBT3904, Q2 2N7002K, Q3 MMBT3904, U1 LTC6994xS6-2, U2 TPS7A2501DRVR, U3 TLV1824, U4 TLV1824

Commit message: autosave 2026-10-20 15:41:55
Parts:
- added G***: BobcatRacing_Logo_15mm, MYLIB:BobcatRacing_Logo_15mm, F.Cu at (178.5, 100.5)
- moved TP4 5.60 mm to (168.0, 94.0)
Other:
- board text added: "This will shutdown the car by december. -RM"

Commit message: autosave 2026-10-21 00:26:08
Parts:
- added TP5: TestPoint, TestPoint:TestPoint_THTPad_D1.0mm_Drill0.5mm, F.Cu at (154.9, 75.2)
- moved G*** 3.02 mm to (179.1, 97.5)
Routing:
- net Latch Input Sensor after 10ms: track 4.24 -> 7.34 mm
Other:
- board text added: "Are you sure its going to work? -CSE"
- board text added: "Relays never win arguments. They always flip. I told a relay my best joke. It didn't laugh, but I could tell it clicked."
- board text added: "TP1: No Fault In Sensor Wiring"
- board text added: "TP2: 5KW Level Demand Reached"
- board text added: "TP3: Brake and 5KW After Delay"
- board text added: "TP4: Ground Point"
- board text added: "TP5: No Fault After 10ms Wire"

Commit message: autosave 2026-10-26 09:17:37
Routing:
- net 5V supply: track 18.4 -> 19.0 mm
- net GND: track 43.0 -> 43.5 mm
Changed lines of the file:
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@@
+	)
+	(segment
+		(start 145.5 86.5)
+		(end 146.148 85.852)
+		(width 0.2)
+		(layer "F.Cu")
+		(net "5V supply")
 	)
 	(segment
@@
 	)
 	(segment
-		(start 147.189 85.475)
-		(end 147.32 85.475)
+		(start 145.288 64.516)
+		(end 147.32 64.516)
 		(width 0.2)
 		(layer "F.Cu")
@@
 	)
 	(segment
-		(start 145.288 64.516)
-		(end 147.32 64.516)
-		(width 0.2)
-		(layer "F.Cu")
-		(net "5V supply")
-	)
-	(segment
 		(start 143.5 73.5)
 		(end 142.3625 73.5)
@@
 	)
 	(segment
-		(start 145.796 85.852)
-		(end 146.812 85.852)
-		(width 0.2)
-		(layer "F.Cu")
-		(net "5V supply")
-	)
-	(segment
 		(start 148.336 79.756)
 		(end 147.828 79.248)
@@
 		(end 142.2625 73.4)
 		(width 0.5)
+		(layer "F.Cu")
+		(net "5V supply")
+	)
+	(segment
+		(start 146.148 85.852)
+		(end 146.812 85.852)
+		(width 0.2)
 		(layer "F.Cu")
 		(net "5V supply")
@@
 	)
 	(segment
+		(start 147.189 85.475)
+		(end 147.32 85.475)
+		(width 0.2)
+		(layer "F.Cu")
+		(net "5V supply")
+	)
+	(segment
 		(start 149.352 79.756)
 		(end 148.336 79.756)
@@
 	)
 	(via
-		(at 145.796 85.852)
+		(at 145.5 86.5)
 		(size 0.6)
 		(drill 0.3)
@@
 		(layer "B.Cu")
 		(net "Net-(R32-Pad2)")
+	)
+	(segment
+		(start 147.75 85)
+		(end 147.8 84.95)
+		(width 0.35)
+		(layer "F.Cu")
+		(net "GND")
 	)
 	(segment
@@
 	)
 	(segment
-		(start 146.5 85)
-		(end 147.75 85)
-		(width 0.35)
-		(layer "F.Cu")
-		(net "GND")
-	)
-	(segment
 		(start 167.5 99.274999)
 		(end 167.5 99.912499)
@@
 		(end 138.176 61.6)
 		(width 0.2)
-		(layer "F.Cu")
-		(net "GND")
-	)
-	(segment
-		(start 147.75 85)
-		(end 147.8 84.95)
-		(width 0.35)
 		(layer "F.Cu")
 		(net "GND")
@@
 	)
 	(segment
+		(start 146 85)
+		(end 147.75 85)
+		(width 0.35)
+		(layer "F.Cu")
+		(net "GND")
+	)
+	(segment
 		(start 160 79.9375)
 		(end 159.95 79.8875)
@@
 	)
 	(via
-		(at 146.5 85)
+		(at 146 85)
 		(size 0.6)
 		(drill 0.3)
@@
 	)
 	(segment
+		(start 151.4125 76)
+		(end 151.4125 77.6955)
+		(width 0.5)
+		(layer "F.Cu")
+		(net "Latch Input Sensor after 10ms")
+	)
+	(segment
+		(start 154 76.124)
+		(end 154.686 75.438)
+		(width 0.2)
+		(layer "F.Cu")
+		(net "Latch Input Sensor after 10ms")
+	)
+	(segment
+		(start 151.5 78.05)
+		(end 153.742 78.05)
+		(width 0.5)
+		(layer "F.Cu")
+		(net "Latch Input Sensor after 10ms")
+	)
+	(segment
+		(start 154 78)
+		(end 154 76.124)
+		(width 0.2)
+		(layer "F.Cu")
+		(net "Latch Input Sensor after 10ms")
+	)
+	(segment
+		(start 154.94 75.184)
+		(end 154.94 75.438)
+		(width 0.2)
+		(layer "F.Cu")
+		(net "Latch Input Sensor after 10ms")
+	)
+	(segment
+		(start 153.742 78.05)
+		(end 153.924 78.232)
+		(width 0.2)
+		(layer "F.Cu")
+		(net "Latch Input Sensor after 10ms")
+	)
+	(segment
+		(start 151.4125 77.6955)
+		(end 151.384 77.724)
+		(width 0.2)
+		(layer "F.Cu")
+		(net "Latch Input Sensor after 10ms")
+	)
+	(segment
 		(start 164.4615 74.0375)
 		(end 164.592 74.168)
@@
 	)
 	(segment
-		(start 151.4125 76)
-		(end 151.4125 77.6955)
-		(width 0.5)
-		(layer "F.Cu")
-		(net "Latch Input Sensor after 10ms")
-	)
-	(segment
-		(start 154 76.124)
-		(end 154.686 75.438)
-		(width 0.2)
-		(layer "F.Cu")
-		(net "Latch Input Sensor after 10ms")
-	)
-	(segment
-		(start 151.5 78.05)
-		(end 153.742 78.05)
-		(width 0.5)
-		(layer "F.Cu")
-		(net "Latch Input Sensor after 10ms")
-	)
-	(segment
-		(start 154 78)
-		(end 154 76.124)
-		(width 0.2)
-		(layer "F.Cu")
-		(net "Latch Input Sensor after 10ms")
-	)
-	(segment
-		(start 154.94 75.184)
-		(end 154.94 75.438)
-		(width 0.2)
-		(layer "F.Cu")
-		(net "Latch Input Sensor after 10ms")
-	)
-	(segment
-		(start 153.742 78.05)
-		(end 153.924 78.232)
-		(width 0.2)
-		(layer "F.Cu")
-		(net "Latch Input Sensor after 10ms")
-	)
-	(segment
-		(start 151.4125 77.6955)
-		(end 151.384 77.724)
-		(width 0.2)
-		(layer "F.Cu")
-		(net "Latch Input Sensor after 10ms")
-	)
-	(segment

Commit message: autosave 2026-10-26 19:41:23
Parts:
- removed J1: 430450412, MYLIB:CONN_SD-43045-005_04_MOL
- added J3: 430450612, MYLIB:CONN_SD-43045-005_06_MOL, F.Cu at (154.5, 101.0)
- moved D1 6.36 mm to (164.0, 95.5)
- moved C10 3.89 mm to (161.0, 98.7)
- moved C12 3.89 mm to (160.9, 102.2)
- moved C13 3.89 mm to (171.5, 103.0)
- moved R4 3.89 mm to (169.0, 99.7)
- moved R5 3.89 mm to (169.0, 103.0)
- moved TP4 3.89 mm to (171.5, 95.7)
- moved U2 3.89 mm to (165.5, 102.2)
- moved G*** 1.43 mm to (180.5, 97.5)
Routing:
- net Vsupply12: track 27.5 -> 32.3 mm
- net GND: track 43.5 -> 44.3 mm, vias 30 -> 29
- net 5kw level: track 57.4 -> 58.2 mm
- net Brake Sensor: track 35.5 -> 36.3 mm

Commit message: autosave 2026-10-26 19:45:43
Routing:
- net GND: track 44.3 -> 47.2 mm, vias 29 -> 30
Changed lines of the file:
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@@
 		(tags "resistor")
 		(property "Reference" "R5"
-			(at -2.4125 -0.500001 0)
+			(at -1.95 -1.999999 0)
 			(layer "F.SilkS")
 			(effects
@@
 		(tags "capacitor")
 		(property "Reference" "C13"
-			(at -2.5 0.499999 180)
+			(at -1.45 2.500001 180)
 			(layer "F.SilkS")
 			(effects
@@
 	)
 	(segment
+		(start 162 91)
+		(end 162.85 90.15)
+		(width 0.8)
+		(layer "F.Cu")
+		(net "GND")
+	)
+	(segment
 		(start 166 100.5)
 		(end 166.578032 101.078032)
@@
 	)
 	(segment
+		(start 162.85 90.15)
+		(end 164 90.15)
+		(width 0.8)
+		(layer "F.Cu")
+		(net "GND")
+	)
+	(segment
 		(start 176.5 81.5)
 		(end 174.9875 81.5)
@@
 	)
 	(segment
+		(start 161.5 91)
+		(end 162 91)
+		(width 0.8)
+		(layer "F.Cu")
+		(net "GND")
+	)
+	(segment
 		(start 136.6725 77.5)
 		(end 136.6725 76.85)
@@
 		(size 0.6)
 		(drill 0.3)
+		(layers "F.Cu" "B.Cu")
+		(free yes)
+		(net "GND")
+	)
+	(via
+		(at 161.5 91)
+		(size 0.6)
+		(drill 0.3)

Commit message: autosave 2026-10-26 20:07:14
Connections:
- C10 pad 2: GND -> Current Sensor -
- C11 pad 2: GND -> Current Sensor -
- C12 pad 2: GND -> Current Sensor -
- C13 pad 2: GND -> Current Sensor -
- C15 pad 2: GND -> Current Sensor -
- C5 pad 2: GND -> Current Sensor -
- C6 pad 2: GND -> Current Sensor -
- C7 pad 2: GND -> Current Sensor -
- C8 pad 2: GND -> Current Sensor -
- C9 pad 1: GND -> Current Sensor -
- CR1 pad 2: GND -> Current Sensor -
- D3 pad 2: GND -> Current Sensor -
- J3 pad 1: unconnected-(J3-Pad1) -> Current Sensor -
- J3 pad 2: unconnected-(J3-Pad2) -> 5V supply
- J3 pad 4: GND -> Current Sensor -
- Q1 pad 2: GND -> Current Sensor -
- Q2 pad 2: GND -> Current Sensor -
- Q3 pad 2: GND -> Current Sensor -
- R10 pad 1: GND -> Current Sensor -
- R11 pad 1: GND -> Current Sensor -
- R13 pad 1: GND -> Current Sensor -
- R17 pad 3: GND -> Current Sensor -
- R19 pad 1: GND -> Current Sensor -
- R2 pad 2: GND -> Current Sensor -
- R22 pad 3: GND -> Current Sensor -
- R26 pad 3: GND -> Current Sensor -
- R27 pad 3: GND -> Current Sensor -
- R3 pad 2: GND -> Current Sensor -
- R32 pad 3: GND -> Current Sensor -
- R33 pad 3: GND -> Current Sensor -
- R34 pad 1: GND -> Current Sensor -
- R4 pad 2: GND -> Current Sensor -
- TP4 pad 1: GND -> Current Sensor -
- U1 pad 2: GND -> Current Sensor -
- U2 pad 3: GND -> Current Sensor -
- U2 pad 5: GND -> Current Sensor -
- U2 pad 7: GND -> Current Sensor -
- U3 pad 11: GND -> Current Sensor -
- U3 pad 12: GND -> Current Sensor -
- U4 pad 11: GND -> Current Sensor -
- U4 pad 12: GND -> Current Sensor -
Routing:
- net Current Sensor -: track 0.00 -> 52.5 mm, vias 0 -> 32
- net GND: track 47.2 -> 0.00 mm, vias 30 -> 0
- net 5V supply: track 19.0 -> 22.5 mm, vias 11 -> 12
- added copper zone on In1.Cu, net Current Sensor -
- removed copper zone on In1.Cu, net GND

Commit message: autosave 2026-10-26 20:48:11
Parts:
- added R21: 10k, Resistor_SMD:R_0805_2012Metric, F.Cu at (130.1, 59.0)
- added R25: 10k, Resistor_SMD:R_0805_2012Metric, F.Cu at (129.5, 68.0)
- added R31: 10k, Resistor_SMD:R_0805_2012Metric, F.Cu at (130.0, 72.5)
- added R41: 10k, Resistor_SMD:R_0805_2012Metric, F.Cu at (130.1, 77.5)
- added R43: 10k, Resistor_SMD:R_0805_2012Metric, F.Cu at (130.0, 81.5)
- added R47: 10k, Resistor_SMD:R_0805_2012Metric, F.Cu at (130.0, 88.5)
- added R48: 10k, Resistor_SMD:R_0805_2012Metric, F.Cu at (130.0, 91.5)
- added R49: 10k, Resistor_SMD:R_0805_2012Metric, F.Cu at (126.6, 104.5)
- added R50: 10k, Resistor_SMD:R_0805_2012Metric, F.Cu at (133.5, 92.5)
- added R51: 10k, Resistor_SMD:R_0805_2012Metric, F.Cu at (132.5, 106.5)
- added R52: 10k, Resistor_SMD:R_0805_2012Metric, F.Cu at (138.0, 92.5)
- added R53: 10k, Resistor_SMD:R_0805_2012Metric, F.Cu at (113.5, 82.3)
- moved R32 2.50 mm to (137.5, 101.5)
- moved R33 2.46 mm to (131.5, 101.5)
Connections:
- R17 pad 1: 5V supply -> Net-(R17-Pad1)
- R17 pad 3: Current Sensor - -> Net-(R17-Pad3)
- R22 pad 1: 5V supply -> Net-(R22-Pad1)
- R22 pad 3: Current Sensor - -> Net-(R22-Pad3)
- R26 pad 1: 5V supply -> Net-(R26-Pad1)
- R26 pad 3: Current Sensor - -> Net-(R26-Pad3)
- R27 pad 1: 5V supply -> Net-(R27-Pad1)
- R27 pad 3: Current Sensor - -> Net-(R27-Pad3)
- R32 pad 1: 5V supply -> Net-(R32-Pad1)
- R32 pad 3: Current Sensor - -> Net-(R32-Pad3)
- R33 pad 1: 5V supply -> Net-(R33-Pad1)
- R33 pad 3: Current Sensor - -> Net-(R33-Pad3)
Routing:
- net Current Sensor -: track 52.5 -> 64.2 mm, vias 32 -> 37
- net 5V supply: track 22.5 -> 33.0 mm, vias 12 -> 18
- net Net-(R33-Pad3): track 0.00 -> 5.79 mm
- net Net-(R26-Pad3): track 0.00 -> 5.78 mm
- net Net-(R17-Pad1): track 0.00 -> 5.59 mm
- net Net-(R26-Pad1): track 0.00 -> 5.09 mm
- net Net-(R17-Pad3): track 0.00 -> 5.09 mm
- net Net-(R27-Pad1): track 0.00 -> 4.88 mm
- net Net-(R22-Pad3): track 0.00 -> 4.39 mm
- net Net-(R22-Pad1): track 0.00 -> 4.27 mm
- net Net-(R27-Pad3): track 0.00 -> 4.09 mm
- net Net-(R33-Pad1): track 0.00 -> 4.05 mm
- net Net-(R32-Pad1): track 0.00 -> 3.72 mm
- net Net-(R27-Pad2): track 39.1 -> 41.4 mm
Other:
- board size 70 x 50.3 mm -> 70 x 52.6 mm

Commit message: autosave 2026-10-27 19:49:44
Parts:
- moved R53 36.6 mm to (141.0, 106.5), turned to 180 degrees
Routing:
- net Net-(R32-Pad3): track 0.00 -> 6.07 mm
- net Current Sensor -: track 64.2 -> 65.7 mm, vias 37 -> 38
